File: brain/hw/BAAAHS-BRN01-E/BAAAHS-BRN01-E.sch (EAGLE design)
At the start: 109 parts, among them J1 USB_MICRO-FCI-USB_MICRO_A_RA, J2 PINHD1X3-20AWG, J3 PINHD1X3-20AWG, J4 PINHD1X10-1X10, J5 RB1-125BAG1A, J7 PINHD1X2-1X02, Q1 MMBT3904, Q2 MMBT3904, U1 SN74LVC1T45-DCK6, U2 ESP32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

Commit message: Updated Brain Controller Rev E files
Reflects feedback from Tom
Parts:
- removed D1: BAT54L, diodes:D_SCHOTTKY-SOT23
Connections:
- net 5V0: no longer D1.C
- net VBUS: no longer D1.A
Other:
- note removed: "Schottky Diode to prevent backflow power into usb"
Changed lines of the file:
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@@
 <part name="V11" library="symbols" deviceset="3V3" device=""/>
 <part name="V12" library="symbols" deviceset="5V0" device=""/>
-<part name="V13" library="symbols" deviceset="5V0" device=""/>
 <part name="GND1" library="symbols" deviceset="GND" device=""/>
 <part name="GND2" library="symbols" deviceset="GND" device=""/>
@@
 <part name="GND26" library="symbols" deviceset="GND" device=""/>
 <part name="GND40" library="symbols" deviceset="GND" device=""/>
-<part name="D1" library="diodes" library_urn="urn:adsk.eagle:library:11609018" deviceset="D_SCHOTTKY" device="-SOT23" package3d_urn="urn:adsk.eagle:package:11609095/2" value="BAT54L"/>
 <part name="C3" library="capacitors" library_urn="urn:adsk.eagle:library:11608356" deviceset="C" device="-C0402" package3d_urn="urn:adsk.eagle:package:11608370/2" technology="-4.7UF_10V_10%" value="4.7uF"/>
 <part name="GND41" library="symbols" deviceset="GND" device=""/>
@@
 <sheet>
 <plain>
-<text x="25.4" y="48.26" size="1.778" layer="97">Schottky Diode to prevent
-backflow power into usb</text>
 <text x="58.42" y="226.06" size="1.778" layer="97" rot="R180" align="center">Normal booting &amp; resetting requires
 IO0 pulled up
@@
 <instance part="V11" gate="G$1" x="368.3" y="68.58" smashed="yes"/>
 <instance part="V12" gate="G$1" x="360.68" y="68.58" smashed="yes"/>
-<instance part="V13" gate="G$1" x="38.1" y="43.18" smashed="yes"/>
 <instance part="GND1" gate="G$1" x="55.88" y="45.72" smashed="yes"/>
 <instance part="GND2" gate="G$1" x="276.86" y="33.02" smashed="yes"/>
@@
 <instance part="GND26" gate="G$1" x="198.12" y="35.56" smashed="yes"/>
 <instance part="GND40" gate="G$1" x="187.96" y="35.56" smashed="yes"/>
-<instance part="D1" gate="G$1" x="38.1" y="35.56" smashed="yes" rot="R90">
-<attribute name="NAME" x="40.132" y="36.449" size="1.778" layer="95"/>
-<attribute name="VALUE" x="40.132" y="33.909" size="1.778" layer="96"/>
-</instance>
 <instance part="C3" gate="G$1" x="50.8" y="20.32" smashed="yes">
 <attribute name="NAME" x="51.816" y="20.955" size="1.778" layer="95"/>
@@
 </segment>
 <segment>
-<pinref part="V13" gate="G$1" pin="5V0"/>
-<pinref part="D1" gate="G$1" pin="C"/>
-<wire x1="38.1" y1="40.64" x2="38.1" y2="38.1" width="0.1524" layer="91"/>
-</segment>
-<segment>
 <pinref part="V25" gate="G$1" pin="5V0"/>
 <pinref part="U7" gate="A" pin="VCCB"/>
@@
 <net name="VBUS" class="0">
 <segment>
-<pinref part="D1" gate="G$1" pin="A"/>
-<wire x1="50.8" y1="30.48" x2="38.1" y2="30.48" width="0.1524" layer="91"/>
-<wire x1="38.1" y1="30.48" x2="35.56" y2="30.48" width="0.1524" layer="91"/>
-<wire x1="38.1" y1="33.02" x2="38.1" y2="30.48" width="0.1524" layer="91"/>
-<junction x="38.1" y="30.48"/>
+<wire x1="50.8" y1="30.48" x2="35.56" y2="30.48" width="0.1524" layer="91"/>
 <pinref part="C3" gate="G$1" pin="1"/>
 <wire x1="50.8" y1="22.86" x2="50.8" y2="30.48" width="0.1524" layer="91"/>

Commit message: Updated Rev E Brain hardware files
Connections:
- net IO39_3V3IO_1_LOW renamed IO39_3V3IO_1_DOWN
Changed lines of the file:
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@@
 </segment>
 </net>
-<net name="IO39_3V3IO_1_LOW" class="0">
+<net name="IO39_3V3IO_1_DOWN" class="0">
 <segment>
 <wire x1="40.64" y1="198.12" x2="15.24" y2="198.12" width="0.1524" layer="91"/>
